File: cw_xcvr/cw_xcvr_kicad/iq_mixer_rx.kicad_sch (KiCad schematic)
At the start: 31 parts, among them Q1 2N3904, Q2 BS170, Q3 2N3904, Q4 BS170, U4 LM324

Commit message: Rx work
Parts:
- removed Q2, Q4: BS170, Package_TO_SOT_THT:TO-92_Inline, symbol Transistor_FET:BS170
- added C10, C8: C, symbol Device:C
- added C11, C9: 160u, symbol Device:C
- added C12: 27n, symbol Device:C
- added L3, L4: 320u, symbol Device:L
- added Q2, Q4: 2N3904, Package_TO_SOT_THT:TO-92_Inline, symbol Transistor_BJT:2N3904
- added R15, R16, R17, R18: R, custom_footprint_library:0.4_pitch_resistor, symbol Device:R
- added R19: 10K, symbol Device:R_Variable_US
- added R20: 2K, custom_footprint_library:0.4_pitch_resistor, symbol Device:R
- added U5, U6: ~, Connector_PinHeader_2.54mm:PinHeader_1x02_P2.54mm_Vertical, symbol custom_symbol_lib:jumper_simple
- C5: value C -> 27n
- R6, R8: value R_Variable_US -> 10K
- R7: value R -> 2K
Connections:
- net GND: now also C3.1, C4.1, R5.2, C10.1, C11.1, C12.2, C8.1, C9.1, L3.1, L4.1, Q2.1 (E), Q4.1 (E), R15.2; no longer Q1.1 (E), Q3.1 (E)
- net Local_osc_I: now also R16.2
- net Local_osc_Q: now also R18.2
- net Power: now also R17.1, R20.1; no longer R2.1, R3.1, R5.1
- net at C5.1, R8.1: now also R19.2; no longer U4.10 (+)
- net at R6.2, R7.1, U4.6 (-): now also R20.2
- net at C3.2: now also L1.2, R2.2; no longer L1.1
- net at R1.2: now also Q1.3 (C), R2.1, C9.2, L3.2, Q2.3 (C), U5.1 (A); no longer C3.1
- net at C2.2, Q3.2 (B): now also L2.1; no longer R3.2
- net at C4.2: now also L2.2, R3.2; no longer L2.1
- net at C1.2, Q1.2 (B): now also L1.1; no longer R2.2
- new net: Q2.2 (B), R16.1
- new net: C10.2, Q3.1 (E), R5.1
- new net: C11.2, L4.2, Q3.3 (C), Q4.3 (C), R17.2, R3.1, U6.1 (A)
- new net: C8.2, Q1.1 (E), R15.1
- new net: C7.1, U6.2 (B)
- new net: C12.1, R19.1, U4.10 (+)
- new net: C6.1, U5.2 (B)
- new net: Q4.2 (B), R18.1
Other:
- note added: "700 Hz filter"
- note added: "90 degree phase shift Adjustable"
- note added: "AC GND"
- note added: "LO shunt, used as a switch"
- note added: "This buffer is given a gain of about 10 to match loss from RC phase shift"
- note removed: "Mixers work by shorting the BJT amplifiers (RF) with the MOSFETs (LO)"
- note removed: "Phase shift adj"
- note removed: "Q Mixer"
- note removed: "Sidetone bandpass"
- note removed: "This buffer is given a bit of gain to match loss from RC phase shift"
- moved on the sheet: C1, C5, C6, Q1, R1, R10, R11, R2, R6, R7, R8, R9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

Commit message: updating computer
Parts:
- added C13: C, symbol Device:C
- added C14: 160u, symbol Device:C
- added C15: 100u, symbol Device:C
- added C16: 20u, symbol Device:C
- added L5: L, symbol Device:L
- added L6: 320u, symbol Device:L
- C11: value 160u -> 100u
- C7: value 20u -> C
- L4: value 320u -> L
- R13, R14: value 10K -> R
- R17, R18: value R -> 10K
Connections:
- net GND: now also C10.2, C7.1, R18.2, C13.2, C14.1, L6.1; no longer C10.1, C11.1, L4.1, R14.2
- net Local_osc_Q: now also R14.2; no longer R18.2
- net at Q3.1 (E), R5.1: now also C7.2; no longer C10.2
- net at U6.2 (B): now also U4.5 (+); no longer C7.1
- net at C6.2, R11.2, R12.1: now also U5.1 (A); no longer U4.3 (+)
- net at C6.1: now also C9.2, L3.2, C15.2; no longer U5.2 (B)
- net at Q4.2 (B): now also R14.1; no longer R18.1
- new net: C15.1, L5.1, Q1.3 (C), Q2.3 (C)
- new net: C11.1, L4.1, Q3.3 (C), Q4.3 (C)
- new net: C13.1, L5.2, R1.2, R2.1
- new net: C16.2, R17.2, R18.1, U6.1 (A)
- new net: U4.3 (+), U5.2 (B)
- new net: C11.2, C14.2, C16.1, L6.2
- new net: C10.1, L4.2, R13.2, R3.1
Other:
- note added: "DC Block"
- note added: "DC Block, set to center of supply for op-amps"
- note added: "Q Mixer"
- note removed: "AC GND"
- note removed: "LPF TC = 100 mS"
- moved on the sheet: C3, C6, C9, L3, R1, R11, R12, R2, R20, R7, U5, U6
